File: pop-badge/rgbleds.sch (KiCad schematic (older format))
At the start: 50 parts, among them U1 WS2812-2020, U10 WS2812-2020, U11 WS2812-2020, U12 WS2812-2020, U13 WS2812-2020, U14 WS2812-2020, U15 WS2812-2020, U16 WS2812-2020, U17 WS2812-2020, U18 WS2812-2020, U19 WS2812-2020, U2 WS2812-2020, U20 WS2812-2020, U21 WS2812-2020, U22 WS2812-2020, U23 WS2812-2020, U24 WS2812-2020, U25 WS2812-2020, U3 WS2812-2020, U4 WS2812-2020, U5 WS2812-2020, U6 WS2812-2020, U7 WS2812-2020, U8 WS2812-2020, U9 WS2812-2020

Commit message: add decoupling cap footprints
Parts:
- C1, C10, C11, C12, C13, C14, C15, C16, C17, C18, C19, C2, C20, C21, C22, C23, C24, C25, C3, C4, C5, C6, C7, C8, C9: footprint (none) -> Capacitor_SMD:C_0603_1608Metric
Changed lines of the file:
@@
 F 0 "C1" V 3350 1150 50  0000 C CNN
 F 1 "100nF" V 3450 1150 50  0000 C CNN
-F 2 "" H 3550 1000 50  0001 C CNN
+F 2 "Capacitor_SMD:C_0603_1608Metric" H 3550 1000 50  0001 C CNN
 F 3 "~" H 3550 1000 50  0001 C CNN
 	1    3550 1000
@@
 F 0 "C3" V 6150 1150 50  0000 C CNN
 F 1 "100nF" V 6250 1150 50  0000 C CNN
-F 2 "" H 6350 1000 50  0001 C CNN
+F 2 "Capacitor_SMD:C_0603_1608Metric" H 6350 1000 50  0001 C CNN
 F 3 "~" H 6350 1000 50  0001 C CNN
 	1    6350 1000
@@
 F 0 "C2" V 4750 1150 50  0000 C CNN
 F 1 "100nF" V 4850 1150 50  0000 C CNN
-F 2 "" H 4950 1000 50  0001 C CNN
+F 2 "Capacitor_SMD:C_0603_1608Metric" H 4950 1000 50  0001 C CNN
 F 3 "~" H 4950 1000 50  0001 C CNN
 	1    4950 1000
@@
 F 0 "C4" V 7550 1150 50  0000 C CNN
 F 1 "100nF" V 7650 1150 50  0000 C CNN
-F 2 "" H 7750 1000 50  0001 C CNN
+F 2 "Capacitor_SMD:C_0603_1608Metric" H 7750 1000 50  0001 C CNN
 F 3 "~" H 7750 1000 50  0001 C CNN
 	1    7750 1000
@@
 F 0 "C5" V 8950 1150 50  0000 C CNN
 F 1 "100nF" V 9050 1150 50  0000 C CNN
-F 2 "" H 9150 1000 50  0001 C CNN
+F 2 "Capacitor_SMD:C_0603_1608Metric" H 9150 1000 50  0001 C CNN
 F 3 "~" H 9150 1000 50  0001 C CNN
 	1    9150 1000
@@
 F 0 "C10" V 8950 2400 50  0000 C CNN
 F 1 "100nF" V 9050 2400 50  0000 C CNN
-F 2 "" H 9150 2250 50  0001 C CNN
+F 2 "Capacitor_SMD:C_0603_1608Metric" H 9150 2250 50  0001 C CNN
 F 3 "~" H 9150 2250 50  0001 C CNN
 	1    9150 2250
@@
 F 0 "C9" V 7550 2400 50  0000 C CNN
 F 1 "100nF" V 7650 2400 50  0000 C CNN
-F 2 "" H 7750 2250 50  0001 C CNN
+F 2 "Capacitor_SMD:C_0603_1608Metric" H 7750 2250 50  0001 C CNN
 F 3 "~" H 7750 2250 50  0001 C CNN
 	1    7750 2250
@@
 F 0 "C8" V 6150 2400 50  0000 C CNN
 F 1 "100nF" V 6250 2400 50  0000 C CNN
-F 2 "" H 6350 2250 50  0001 C CNN
+F 2 "Capacitor_SMD:C_0603_1608Metric" H 6350 2250 50  0001 C CNN
 F 3 "~" H 6350 2250 50  0001 C CNN
 	1    6350 2250
@@
 F 0 "C7" V 4750 2400 50  0000 C CNN
 F 1 "100nF" V 4850 2400 50  0000 C CNN
-F 2 "" H 4950 2250 50  0001 C CNN
+F 2 "Capacitor_SMD:C_0603_1608Metric" H 4950 2250 50  0001 C CNN
 F 3 "~" H 4950 2250 50  0001 C CNN
 	1    4950 2250
@@
 F 0 "C12" V 4750 3600 50  0000 C CNN
 F 1 "100nF" V 4850 3600 50  0000 C CNN
-F 2 "" H 4950 3450 50  0001 C CNN
+F 2 "Capacitor_SMD:C_0603_1608Metric" H 4950 3450 50  0001 C CNN
 F 3 "~" H 4950 3450 50  0001 C CNN
 	1    4950 3450
@@
 F 0 "C13" V 6150 3600 50  0000 C CNN
 F 1 "100nF" V 6250 3600 50  0000 C CNN
-F 2 "" H 6350 3450 50  0001 C CNN
+F 2 "Capacitor_SMD:C_0603_1608Metric" H 6350 3450 50  0001 C CNN
 F 3 "~" H 6350 3450 50  0001 C CNN
 	1    6350 3450
@@
 F 0 "C14" V 7550 3600 50  0000 C CNN
 F 1 "100nF" V 7650 3600 50  0000 C CNN
-F 2 "" H 7750 3450 50  0001 C CNN
+F 2 "Capacitor_SMD:C_0603_1608Metric" H 7750 3450 50  0001 C CNN
 F 3 "~" H 7750 3450 50  0001 C CNN
 	1    7750 3450
@@
 F 0 "C15" V 8950 3600 50  0000 C CNN
 F 1 "100nF" V 9050 3600 50  0000 C CNN
-F 2 "" H 9150 3450 50  0001 C CNN
+F 2 "Capacitor_SMD:C_0603_1608Metric" H 9150 3450 50  0001 C CNN
 F 3 "~" H 9150 3450 50  0001 C CNN
 	1    9150 3450
@@
 F 0 "C6" V 3350 2400 50  0000 C CNN
 F 1 "100nF" V 3450 2400 50  0000 C CNN
-F 2 "" H 3550 2250 50  0001 C CNN
+F 2 "Capacitor_SMD:C_0603_1608Metric" H 3550 2250 50  0001 C CNN
 F 3 "~" H 3550 2250 50  0001 C CNN
 	1    3550 2250
@@
 F 0 "C11" V 3350 3600 50  0000 C CNN
 F 1 "100nF" V 3450 3600 50  0000 C CNN
-F 2 "" H 3550 3450 50  0001 C CNN
+F 2 "Capacitor_SMD:C_0603_1608Metric" H 3550 3450 50  0001 C CNN
 F 3 "~" H 3550 3450 50  0001 C CNN
 	1    3550 3450
@@
 F 0 "C25" V 8950 5900 50  0000 C CNN
 F 1 "100nF" V 9050 5900 50  0000 C CNN
-F 2 "" H 9150 5750 50  0001 C CNN
+F 2 "Capacitor_SMD:C_0603_1608Metric" H 9150 5750 50  0001 C CNN
 F 3 "~" H 9150 5750 50  0001 C CNN
 	1    9150 5750
@@
 F 0 "C20" V 8950 4750 50  0000 C CNN
 F 1 "100nF" V 9050 4750 50  0000 C CNN
-F 2 "" H 9150 4600 50  0001 C CNN
+F 2 "Capacitor_SMD:C_0603_1608Metric" H 9150 4600 50  0001 C CNN
 F 3 "~" H 9150 4600 50  0001 C CNN
 	1    9150 4600
@@
 F 0 "C19" V 7550 4750 50  0000 C CNN
 F 1 "100nF" V 7650 4750 50  0000 C CNN
-F 2 "" H 7750 4600 50  0001 C CNN
+F 2 "Capacitor_SMD:C_0603_1608Metric" H 7750 4600 50  0001 C CNN
 F 3 "~" H 7750 4600 50  0001 C CNN
 	1    7750 4600
@@
 F 0 "C18" V 6150 4750 50  0000 C CNN
 F 1 "100nF" V 6250 4750 50  0000 C CNN
-F 2 "" H 6350 4600 50  0001 C CNN
+F 2 "Capacitor_SMD:C_0603_1608Metric" H 6350 4600 50  0001 C CNN
 F 3 "~" H 6350 4600 50  0001 C CNN
 	1    6350 4600
@@
 F 0 "C24" V 7550 5900 50  0000 C CNN
 F 1 "100nF" V 7650 5900 50  0000 C CNN
-F 2 "" H 7750 5750 50  0001 C CNN
+F 2 "Capacitor_SMD:C_0603_1608Metric" H 7750 5750 50  0001 C CNN
 F 3 "~" H 7750 5750 50  0001 C CNN
 	1    7750 5750
@@
 F 0 "C23" V 6150 5900 50  0000 C CNN
 F 1 "100nF" V 6250 5900 50  0000 C CNN
-F 2 "" H 6350 5750 50  0001 C CNN
+F 2 "Capacitor_SMD:C_0603_1608Metric" H 6350 5750 50  0001 C CNN
 F 3 "~" H 6350 5750 50  0001 C CNN
 	1    6350 5750
@@
 F 0 "C22" V 4750 5900 50  0000 C CNN
 F 1 "100nF" V 4850 5900 50  0000 C CNN
-F 2 "" H 4950 5750 50  0001 C CNN
+F 2 "Capacitor_SMD:C_0603_1608Metric" H 4950 5750 50  0001 C CNN
 F 3 "~" H 4950 5750 50  0001 C CNN
 	1    4950 5750
@@
 F 0 "C21" V 3350 5900 50  0000 C CNN
 F 1 "100nF" V 3450 5900 50  0000 C CNN
-F 2 "" H 3550 5750 50  0001 C CNN
+F 2 "Capacitor_SMD:C_0603_1608Metric" H 3550 5750 50  0001 C CNN
 F 3 "~" H 3550 5750 50  0001 C CNN
 	1    3550 5750
@@
 F 0 "C16" V 3350 4750 50  0000 C CNN
 F 1 "100nF" V 3450 4750 50  0000 C CNN
-F 2 "" H 3550 4600 50  0001 C CNN
+F 2 "Capacitor_SMD:C_0603_1608Metric" H 3550 4600 50  0001 C CNN
 F 3 "~" H 3550 4600 50  0001 C CNN
 	1    3550 4600
@@
 F 0 "C17" V 4750 4750 50  0000 C CNN
 F 1 "100nF" V 4850 4750 50  0000 C CNN
-F 2 "" H 4950 4600 50  0001 C CNN
+F 2 "Capacitor_SMD:C_0603_1608Metric" H 4950 4600 50  0001 C CNN
 F 3 "~" H 4950 4600 50  0001 C CNN
 	1    4950 4600

Commit message: routing done
Parts:
- added C26: 100u, Capacitor_THT:CP_Radial_D6.3mm_P2.50mm, symbol Device:CP
- added R52: 220R, Resistor_SMD:R_0603_1608Metric_Pad1.05x0.95mm_HandSolder, symbol Device:R
- C1, C10, C11, C12, C13, C14, C15, C16, C17, C18, C19, C2, C20, C21, C22, C23, C24, C25, C3, C4, C5, C6, C7, C8, C9: footprint Capacitor_SMD:C_0603_1608Metric -> Capacitor_SMD:C_0402_1005Metric
Connections:
- net +5V: now also C26.1
- net DIN: now also R52.2; no longer U1.3 (DI)
- net GND: now also C26.2
- new net: R52.1, U1.3 (DI)
Changed lines of the file:
@@
 $Descr A4 11693 8268
 encoding utf-8
-Sheet 3 3
+Sheet 2 3
 Title ""
 Date ""
@@
 DIN
 Wire Wire Line
-	1300 1200 2250 1200
-Wire Wire Line
 	1300 900  1450 900
 Wire Wire Line
@@
 F 0 "C1" V 3350 1150 50  0000 C CNN
 F 1 "100nF" V 3450 1150 50  0000 C CNN
-F 2 "Capacitor_SMD:C_0603_1608Metric" H 3550 1000 50  0001 C CNN
+F 2 "Capacitor_SMD:C_0402_1005Metric" H 3550 1000 50  0001 C CNN
 F 3 "~" H 3550 1000 50  0001 C CNN
 	1    3550 1000
@@
 F 0 "C3" V 6150 1150 50  0000 C CNN
 F 1 "100nF" V 6250 1150 50  0000 C CNN
-F 2 "Capacitor_SMD:C_0603_1608Metric" H 6350 1000 50  0001 C CNN
+F 2 "Capacitor_SMD:C_0402_1005Metric" H 6350 1000 50  0001 C CNN
 F 3 "~" H 6350 1000 50  0001 C CNN
 	1    6350 1000
@@
 F 0 "C2" V 4750 1150 50  0000 C CNN
 F 1 "100nF" V 4850 1150 50  0000 C CNN
-F 2 "Capacitor_SMD:C_0603_1608Metric" H 4950 1000 50  0001 C CNN
+F 2 "Capacitor_SMD:C_0402_1005Metric" H 4950 1000 50  0001 C CNN
 F 3 "~" H 4950 1000 50  0001 C CNN
 	1    4950 1000
@@
 F 0 "C4" V 7550 1150 50  0000 C CNN
 F 1 "100nF" V 7650 1150 50  0000 C CNN
-F 2 "Capacitor_SMD:C_0603_1608Metric" H 7750 1000 50  0001 C CNN
+F 2 "Capacitor_SMD:C_0402_1005Metric" H 7750 1000 50  0001 C CNN
 F 3 "~" H 7750 1000 50  0001 C CNN
 	1    7750 1000
@@
 F 0 "C5" V 8950 1150 50  0000 C CNN
 F 1 "100nF" V 9050 1150 50  0000 C CNN
-F 2 "Capacitor_SMD:C_0603_1608Metric" H 9150 1000 50  0001 C CNN
+F 2 "Capacitor_SMD:C_0402_1005Metric" H 9150 1000 50  0001 C CNN
 F 3 "~" H 9150 1000 50  0001 C CNN
 	1    9150 1000
@@
 F 0 "C10" V 8950 2400 50  0000 C CNN
 F 1 "100nF" V 9050 2400 50  0000 C CNN
-F 2 "Capacitor_SMD:C_0603_1608Metric" H 9150 2250 50  0001 C CNN
+F 2 "Capacitor_SMD:C_0402_1005Metric" H 9150 2250 50  0001 C CNN
 F 3 "~" H 9150 2250 50  0001 C CNN
 	1    9150 2250
@@
 F 0 "C9" V 7550 2400 50  0000 C CNN
 F 1 "100nF" V 7650 2400 50  0000 C CNN
-F 2 "Capacitor_SMD:C_0603_1608Metric" H 7750 2250 50  0001 C CNN
+F 2 "Capacitor_SMD:C_0402_1005Metric" H 7750 2250 50  0001 C CNN
 F 3 "~" H 7750 2250 50  0001 C CNN
 	1    7750 2250
@@
 F 0 "C8" V 6150 2400 50  0000 C CNN
 F 1 "100nF" V 6250 2400 50  0000 C CNN
-F 2 "Capacitor_SMD:C_0603_1608Metric" H 6350 2250 50  0001 C CNN
+F 2 "Capacitor_SMD:C_0402_1005Metric" H 6350 2250 50  0001 C CNN
 F 3 "~" H 6350 2250 50  0001 C CNN
 	1    6350 2250
@@
 F 0 "C7" V 4750 2400 50  0000 C CNN
 F 1 "100nF" V 4850 2400 50  0000 C CNN
-F 2 "Capacitor_SMD:C_0603_1608Metric" H 4950 2250 50  0001 C CNN
+F 2 "Capacitor_SMD:C_0402_1005Metric" H 4950 2250 50  0001 C CNN
 F 3 "~" H 4950 2250 50  0001 C CNN
 	1    4950 2250
@@
 F 0 "C12" V 4750 3600 50  0000 C CNN
 F 1 "100nF" V 4850 3600 50  0000 C CNN
-F 2 "Capacitor_SMD:C_0603_1608Metric" H 4950 3450 50  0001 C CNN
+F 2 "Capacitor_SMD:C_0402_1005Metric" H 4950 3450 50  0001 C CNN
 F 3 "~" H 4950 3450 50  0001 C CNN
 	1    4950 3450
@@
 F 0 "C13" V 6150 3600 50  0000 C CNN
 F 1 "100nF" V 6250 3600 50  0000 C CNN
-F 2 "Capacitor_SMD:C_0603_1608Metric" H 6350 3450 50  0001 C CNN
+F 2 "Capacitor_SMD:C_0402_1005Metric" H 6350 3450 50  0001 C CNN
 F 3 "~" H 6350 3450 50  0001 C CNN
 	1    6350 3450
@@
 F 0 "C14" V 7550 3600 50  0000 C CNN
 F 1 "100nF" V 7650 3600 50  0000 C CNN
-F 2 "Capacitor_SMD:C_0603_1608Metric" H 7750 3450 50  0001 C CNN
+F 2 "Capacitor_SMD:C_0402_1005Metric" H 7750 3450 50  0001 C CNN
 F 3 "~" H 7750 3450 50  0001 C CNN
 	1    7750 3450
@@
 F 0 "C15" V 8950 3600 50  0000 C CNN
 F 1 "100nF" V 9050 3600 50  0000 C CNN
-F 2 "Capacitor_SMD:C_0603_1608Metric" H 9150 3450 50  0001 C CNN
+F 2 "Capacitor_SMD:C_0402_1005Metric" H 9150 3450 50  0001 C CNN
 F 3 "~" H 9150 3450 50  0001 C CNN
 	1    9150 3450
@@
 F 0 "C6" V 3350 2400 50  0000 C CNN
 F 1 "100nF" V 3450 2400 50  0000 C CNN
-F 2 "Capacitor_SMD:C_0603_1608Metric" H 3550 2250 50  0001 C CNN
+F 2 "Capacitor_SMD:C_0402_1005Metric" H 3550 2250 50  0001 C CNN
 F 3 "~" H 3550 2250 50  0001 C CNN
 	1    3550 2250
@@
 F 0 "C11" V 3350 3600 50  0000 C CNN
 F 1 "100nF" V 3450 3600 50  0000 C CNN
-F 2 "Capacitor_SMD:C_0603_1608Metric" H 3550 3450 50  0001 C CNN
+F 2 "Capacitor_SMD:C_0402_1005Metric" H 3550 3450 50  0001 C CNN
 F 3 "~" H 3550 3450 50  0001 C CNN
 	1    3550 3450
@@
 F 0 "C25" V 8950 5900 50  0000 C CNN
 F 1 "100nF" V 9050 5900 50  0000 C CNN
-F 2 "Capacitor_SMD:C_0603_1608Metric" H 9150 5750 50  0001 C CNN
+F 2 "Capacitor_SMD:C_0402_1005Metric" H 9150 5750 50  0001 C CNN
 F 3 "~" H 9150 5750 50  0001 C CNN
 	1    9150 5750
@@
 F 0 "C20" V 8950 4750 50  0000 C CNN
 F 1 "100nF" V 9050 4750 50  0000 C CNN
-F 2 "Capacitor_SMD:C_0603_1608Metric" H 9150 4600 50  0001 C CNN
+F 2 "Capacitor_SMD:C_0402_1005Metric" H 9150 4600 50  0001 C CNN
 F 3 "~" H 9150 4600 50  0001 C CNN
 	1    9150 4600
@@
 F 0 "C19" V 7550 4750 50  0000 C CNN
 F 1 "100nF" V 7650 4750 50  0000 C CNN
-F 2 "Capacitor_SMD:C_0603_1608Metric" H 7750 4600 50  0001 C CNN
+F 2 "Capacitor_SMD:C_0402_1005Metric" H 7750 4600 50  0001 C CNN
 F 3 "~" H 7750 4600 50  0001 C CNN
 	1    7750 4600
@@
 F 0 "C18" V 6150 4750 50  0000 C CNN
 F 1 "100nF" V 6250 4750 50  0000 C CNN
-F 2 "Capacitor_SMD:C_0603_1608Metric" H 6350 4600 50  0001 C CNN
+F 2 "Capacitor_SMD:C_0402_1005Metric" H 6350 4600 50  0001 C CNN
 F 3 "~" H 6350 4600 50  0001 C CNN
 	1    6350 4600
@@
 F 0 "C24" V 7550 5900 50  0000 C CNN
 F 1 "100nF" V 7650 5900 50  0000 C CNN
-F 2 "Capacitor_SMD:C_0603_1608Metric" H 7750 5750 50  0001 C CNN
+F 2 "Capacitor_SMD:C_0402_1005Metric" H 7750 5750 50  0001 C CNN
 F 3 "~" H 7750 5750 50  0001 C CNN
 	1    7750 5750
@@
 F 0 "C23" V 6150 5900 50  0000 C CNN
 F 1 "100nF" V 6250 5900 50  0000 C CNN
-F 2 "Capacitor_SMD:C_0603_1608Metric" H 6350 5750 50  0001 C CNN
+F 2 "Capacitor_SMD:C_0402_1005Metric" H 6350 5750 50  0001 C CNN
 F 3 "~" H 6350 5750 50  0001 C CNN
 	1    6350 5750
@@
 F 0 "C22" V 4750 5900 50  0000 C CNN
 F 1 "100nF" V 4850 5900 50  0000 C CNN
-F 2 "Capacitor_SMD:C_0603_1608Metric" H 4950 5750 50  0001 C CNN
+F 2 "Capacitor_SMD:C_0402_1005Metric" H 4950 5750 50  0001 C CNN
 F 3 "~" H 4950 5750 50  0001 C CNN
 	1    4950 5750
@@
 F 0 "C21" V 3350 5900 50  0000 C CNN
 F 1 "100nF" V 3450 5900 50  0000 C CNN
-F 2 "Capacitor_SMD:C_0603_1608Metric" H 3550 5750 50  0001 C CNN
+F 2 "Capacitor_SMD:C_0402_1005Metric" H 3550 5750 50  0001 C CNN
 F 3 "~" H 3550 5750 50  0001 C CNN
 	1    3550 5750
@@
 F 0 "C16" V 3350 4750 50  0000 C CNN
 F 1 "100nF" V 3450 4750 50  0000 C CNN
-F 2 "Capacitor_SMD:C_0603_1608Metric" H 3550 4600 50  0001 C CNN
+F 2 "Capacitor_SMD:C_0402_1005Metric" H 3550 4600 50  0001 C CNN
 F 3 "~" H 3550 4600 50  0001 C CNN
 	1    3550 4600
@@
 F 0 "C17" V 4750 4750 50  0000 C CNN
 F 1 "100nF" V 4850 4750 50  0000 C CNN
-F 2 "Capacitor_SMD:C_0603_1608Metric" H 4950 4600 50  0001 C CNN
+F 2 "Capacitor_SMD:C_0402_1005Metric" H 4950 4600 50  0001 C CNN
 F 3 "~" H 4950 4600 50  0001 C CNN
 	1    4950 4600
@@
 Wire Wire Line
 	5050 5000 4850 5000
+$Comp
+L Device:R R52
+U 1 1 61AA409E
+P 1850 1200
+F 0 "R52" V 1643 1200 50  0000 C CNN
+F 1 "220R" V 1734 1200 50  0000 C CNN
+F 2 "Resistor_SMD:R_0603_1608Metric_Pad1.05x0.95mm_HandSolder" V 1780 1200 50  0001 C CNN
+F 3 "~" H 1850 1200 50  0001 C CNN
+	1    1850 1200
+	0    1    1    0
+$EndComp
+Wire Wire Line
+	2250 1200 2000 1200
+Wire Wire Line
+	1700 1200 1300 1200
+$Comp
+L Device:CP C26
+U 1 1 61AAC781
+P 1150 2200
+F 0 "C26" H 1268 2246 50  0000 L CNN
+F 1 "100u" H 1268 2155 50  0000 L CNN
+F 2 "Capacitor_THT:CP_Radial_D6.3mm_P2.50mm" H 1188 2050 50  0001 C CNN
+F 3 "~" H 1150 2200 50  0001 C CNN
+	1    1150 2200
+	1    0    0    -1
+$EndComp
+$Comp
+L power:+5V #PWR0101
+U 1 1 61AAD818
+P 1150 2050
+F 0 "#PWR0101" H 1150 1900 50  0001 C CNN
+F 1 "+5V" H 1165 2223 50  0000 C CNN
+F 2 "" H 1150 2050 50  0001 C CNN
+F 3 "" H 1150 2050 50  0001 C CNN
+	1    1150 2050
+	1    0    0    -1
+$EndComp
+$Comp
+L power:GND #PWR0102
+U 1 1 61AAE140
+P 1150 2350
+F 0 "#PWR0102" H 1150 2100 50  0001 C CNN
+F 1 "GND" H 1155 2177 50  0000 C CNN
+F 2 "" H 1150 2350 50  0001 C CNN
+F 3 "" H 1150 2350 50  0001 C CNN
+	1    1150 2350
+	1    0    0    -1
+$EndComp
 $EndSCHEMATC

Commit message: small bom fixes
Parts:
- C1, C10, C11, C12, C13, C14, C15, C16, C17, C18, C19, C2, C20, C21, C22, C23, C24, C25, C3, C4, C5, C6, C7, C8, C9: JLC (none) -> 0402
- R52: JLC (none) -> 0603
Changed lines of the file:
@@
 F 2 "Capacitor_SMD:C_0402_1005Metric" H 3550 1000 50  0001 C CNN
 F 3 "~" H 3550 1000 50  0001 C CNN
+F 4 "0402" H 3550 1000 50  0001 C CNN "JLC"
 	1    3550 1000
 	0    1    1    0
@@
 F 2 "Capacitor_SMD:C_0402_1005Metric" H 6350 1000 50  0001 C CNN
 F 3 "~" H 6350 1000 50  0001 C CNN
+F 4 "0402" H 6350 1000 50  0001 C CNN "JLC"
 	1    6350 1000
 	0    1    1    0
@@
 F 2 "Capacitor_SMD:C_0402_1005Metric" H 4950 1000 50  0001 C CNN
 F 3 "~" H 4950 1000 50  0001 C CNN
+F 4 "0402" H 4950 1000 50  0001 C CNN "JLC"
 	1    4950 1000
 	0    1    1    0
@@
 F 2 "Capacitor_SMD:C_0402_1005Metric" H 7750 1000 50  0001 C CNN
 F 3 "~" H 7750 1000 50  0001 C CNN
+F 4 "0402" H 7750 1000 50  0001 C CNN "JLC"
 	1    7750 1000
 	0    1    1    0
@@
 F 2 "Capacitor_SMD:C_0402_1005Metric" H 9150 1000 50  0001 C CNN
 F 3 "~" H 9150 1000 50  0001 C CNN
+F 4 "0402" H 9150 1000 50  0001 C CNN "JLC"
 	1    9150 1000
 	0    1    1    0
@@
 F 2 "Capacitor_SMD:C_0402_1005Metric" H 9150 2250 50  0001 C CNN
 F 3 "~" H 9150 2250 50  0001 C CNN
+F 4 "0402" H 9150 2250 50  0001 C CNN "JLC"
 	1    9150 2250
 	0    1    1    0
@@
 F 2 "Capacitor_SMD:C_0402_1005Metric" H 7750 2250 50  0001 C CNN
 F 3 "~" H 7750 2250 50  0001 C CNN
+F 4 "0402" H 7750 2250 50  0001 C CNN "JLC"
 	1    7750 2250
 	0    1    1    0
@@
 F 2 "Capacitor_SMD:C_0402_1005Metric" H 6350 2250 50  0001 C CNN
 F 3 "~" H 6350 2250 50  0001 C CNN
+F 4 "0402" H 6350 2250 50  0001 C CNN "JLC"
 	1    6350 2250
 	0    1    1    0
@@
 F 2 "Capacitor_SMD:C_0402_1005Metric" H 4950 2250 50  0001 C CNN
 F 3 "~" H 4950 2250 50  0001 C CNN
+F 4 "0402" H 4950 2250 50  0001 C CNN "JLC"
 	1    4950 2250
 	0    1    1    0
@@
 F 2 "Capacitor_SMD:C_0402_1005Metric" H 4950 3450 50  0001 C CNN
 F 3 "~" H 4950 3450 50  0001 C CNN
+F 4 "0402" H 4950 3450 50  0001 C CNN "JLC"
 	1    4950 3450
 	0    1    1    0
@@
 F 2 "Capacitor_SMD:C_0402_1005Metric" H 6350 3450 50  0001 C CNN
 F 3 "~" H 6350 3450 50  0001 C CNN
+F 4 "0402" H 6350 3450 50  0001 C CNN "JLC"
 	1    6350 3450
 	0    1    1    0
@@
 F 2 "Capacitor_SMD:C_0402_1005Metric" H 7750 3450 50  0001 C CNN
 F 3 "~" H 7750 3450 50  0001 C CNN
+F 4 "0402" H 7750 3450 50  0001 C CNN "JLC"
 	1    7750 3450
 	0    1    1    0
@@
 F 2 "Capacitor_SMD:C_0402_1005Metric" H 9150 3450 50  0001 C CNN
 F 3 "~" H 9150 3450 50  0001 C CNN
+F 4 "0402" H 9150 3450 50  0001 C CNN "JLC"
 	1    9150 3450
 	0    1    1    0
@@
 F 2 "Capacitor_SMD:C_0402_1005Metric" H 3550 2250 50  0001 C CNN
 F 3 "~" H 3550 2250 50  0001 C CNN
+F 4 "0402" H 3550 2250 50  0001 C CNN "JLC"
 	1    3550 2250
 	0    1    1    0
@@
 F 2 "Capacitor_SMD:C_0402_1005Metric" H 3550 3450 50  0001 C CNN
 F 3 "~" H 3550 3450 50  0001 C CNN
+F 4 "0402" H 3550 3450 50  0001 C CNN "JLC"
 	1    3550 3450
 	0    1    1    0
@@
 F 2 "Capacitor_SMD:C_0402_1005Metric" H 9150 5750 50  0001 C CNN
 F 3 "~" H 9150 5750 50  0001 C CNN
+F 4 "0402" H 9150 5750 50  0001 C CNN "JLC"
 	1    9150 5750
 	0    1    1    0
@@
 F 2 "Capacitor_SMD:C_0402_1005Metric" H 9150 4600 50  0001 C CNN
 F 3 "~" H 9150 4600 50  0001 C CNN
+F 4 "0402" H 9150 4600 50  0001 C CNN "JLC"
 	1    9150 4600
 	0    1    1    0
@@
 F 2 "Capacitor_SMD:C_0402_1005Metric" H 7750 4600 50  0001 C CNN
 F 3 "~" H 7750 4600 50  0001 C CNN
+F 4 "0402" H 7750 4600 50  0001 C CNN "JLC"
 	1    7750 4600
 	0    1    1    0
@@
 F 2 "Capacitor_SMD:C_0402_1005Metric" H 6350 4600 50  0001 C CNN
 F 3 "~" H 6350 4600 50  0001 C CNN
+F 4 "0402" H 6350 4600 50  0001 C CNN "JLC"
 	1    6350 4600
 	0    1    1    0
@@
 F 2 "Capacitor_SMD:C_0402_1005Metric" H 7750 5750 50  0001 C CNN
 F 3 "~" H 7750 5750 50  0001 C CNN
+F 4 "0402" H 7750 5750 50  0001 C CNN "JLC"
 	1    7750 5750
 	0    1    1    0
@@
 F 2 "Capacitor_SMD:C_0402_1005Metric" H 6350 5750 50  0001 C CNN
 F 3 "~" H 6350 5750 50  0001 C CNN
+F 4 "0402" H 6350 5750 50  0001 C CNN "JLC"
 	1    6350 5750
 	0    1    1    0
@@
 F 2 "Capacitor_SMD:C_0402_1005Metric" H 4950 5750 50  0001 C CNN
 F 3 "~" H 4950 5750 50  0001 C CNN
+F 4 "0402" H 4950 5750 50  0001 C CNN "JLC"
 	1    4950 5750
 	0    1    1    0
@@
 F 2 "Capacitor_SMD:C_0402_1005Metric" H 3550 5750 50  0001 C CNN
 F 3 "~" H 3550 5750 50  0001 C CNN
+F 4 "0402" H 3550 5750 50  0001 C CNN "JLC"
 	1    3550 5750
 	0    1    1    0
@@
 F 2 "Capacitor_SMD:C_0402_1005Metric" H 3550 4600 50  0001 C CNN
 F 3 "~" H 3550 4600 50  0001 C CNN
+F 4 "0402" H 3550 4600 50  0001 C CNN "JLC"
 	1    3550 4600
 	0    1    1    0
@@
 F 2 "Capacitor_SMD:C_0402_1005Metric" H 4950 4600 50  0001 C CNN
 F 3 "~" H 4950 4600 50  0001 C CNN
+F 4 "0402" H 4950 4600 50  0001 C CNN "JLC"
 	1    4950 4600
 	0    1    1    0
@@
 F 2 "Resistor_SMD:R_0603_1608Metric_Pad1.05x0.95mm_HandSolder" V 1780 1200 50  0001 C CNN
 F 3 "~" H 1850 1200 50  0001 C CNN
+F 4 "0603" H 1850 1200 50  0001 C CNN "JLC"
 	1    1850 1200
 	0    1    1    0

Commit message: add alternative path
Parts:
- R52: value 220R -> 200
Changed lines of the file:
@@
 $Descr A4 11693 8268
 encoding utf-8
-Sheet 2 3
+Sheet 3 3
 Title ""
 Date ""
@@
 P 1850 1200
 F 0 "R52" V 1643 1200 50  0000 C CNN
-F 1 "220R" V 1734 1200 50  0000 C CNN
+F 1 "200" V 1734 1200 50  0000 C CNN
 F 2 "Resistor_SMD:R_0603_1608Metric_Pad1.05x0.95mm_HandSolder" V 1780 1200 50  0001 C CNN
 F 3 "~" H 1850 1200 50  0001 C CNN
