File: pop-badge/rgbleds.sch (KiCad schematic (older format))
At the start: 52 parts, among them U1 WS2812-2020, U10 WS2812-2020, U11 WS2812-2020, U12 WS2812-2020, U13 WS2812-2020, U14 WS2812-2020, U15 WS2812-2020, U16 WS2812-2020, U17 WS2812-2020, U18 WS2812-2020, U19 WS2812-2020, U2 WS2812-2020, U20 WS2812-2020, U21 WS2812-2020, U22 WS2812-2020, U23 WS2812-2020, U24 WS2812-2020, U25 WS2812-2020, U3 WS2812-2020, U4 WS2812-2020, U5 WS2812-2020, U6 WS2812-2020, U7 WS2812-2020, U8 WS2812-2020, U9 WS2812-2020

Commit message: add rescue lib
Parts:
- U1, U10, U11, U12, U13, U14, U15, U16, U17, U18, U19, U2, U20, U21, U22, U23, U24, U25, U3, U4, U5, U6, U7, U8, U9: symbol WS2812-2020:WS2812-2020 -> pop-badge-rescue:WS2812-2020-WS2812-2020
Changed lines of the file:
@@
 $EndComp
 $Comp
-L WS2812-2020:WS2812-2020 U?
+L pop-badge-rescue:WS2812-2020-WS2812-2020 U?
 U 1 1 617E18CF
 P 2850 1200
@@
 	6250 1200 6450 1200
 $Comp
-L WS2812-2020:WS2812-2020 U?
+L pop-badge-rescue:WS2812-2020-WS2812-2020 U?
 U 1 1 617E18F9
 P 5650 1200
@@
 $EndComp
 $Comp
-L WS2812-2020:WS2812-2020 U?
+L pop-badge-rescue:WS2812-2020-WS2812-2020 U?
 U 1 1 617E190D
 P 7050 1200
@@
 	3450 2450 3650 2450
 $Comp
-L WS2812-2020:WS2812-2020 U?
+L pop-badge-rescue:WS2812-2020-WS2812-2020 U?
 U 1 1 617E37B7
 P 2850 2450
@@
 	4850 2450 5050 2450
 $Comp
-L WS2812-2020:WS2812-2020 U?
+L pop-badge-rescue:WS2812-2020-WS2812-2020 U?
 U 1 1 617E37D8
 P 4250 2450
@@
 	6250 2450 6450 2450
 $Comp
-L WS2812-2020:WS2812-2020 U?
+L pop-badge-rescue:WS2812-2020-WS2812-2020 U?
 U 1 1 617E37F9
 P 5650 2450
@@
 $EndComp
 $Comp
-L WS2812-2020:WS2812-2020 U?
+L pop-badge-rescue:WS2812-2020-WS2812-2020 U?
 U 1 1 617E3819
 P 7050 2450
@@
 $EndComp
 $Comp
-L WS2812-2020:WS2812-2020 U?
+L pop-badge-rescue:WS2812-2020-WS2812-2020 U?
 U 1 1 617E383C
 P 8450 2450
@@
 	3450 3650 3650 3650
 $Comp
-L WS2812-2020:WS2812-2020 U?
+L pop-badge-rescue:WS2812-2020-WS2812-2020 U?
 U 1 1 617EC540
 P 2850 3650
@@
 	4850 3650 5050 3650
 $Comp
-L WS2812-2020:WS2812-2020 U?
+L pop-badge-rescue:WS2812-2020-WS2812-2020 U?
 U 1 1 617EC555
 P 4250 3650
@@
 	6250 3650 6450 3650
 $Comp
-L WS2812-2020:WS2812-2020 U?
+L pop-badge-rescue:WS2812-2020-WS2812-2020 U?
 U 1 1 617EC56A
 P 5650 3650
@@
 $EndComp
 $Comp
-L WS2812-2020:WS2812-2020 U?
+L pop-badge-rescue:WS2812-2020-WS2812-2020 U?
 U 1 1 617EC57E
 P 7050 3650
@@
 $EndComp
 $Comp
-L WS2812-2020:WS2812-2020 U?
+L pop-badge-rescue:WS2812-2020-WS2812-2020 U?
 U 1 1 617EC595
 P 8450 3650
@@
 	3450 4800 3650 4800
 $Comp
-L WS2812-2020:WS2812-2020 U?
+L pop-badge-rescue:WS2812-2020-WS2812-2020 U?
 U 1 1 617EF6EF
 P 2850 4800
@@
 	4850 4800 5050 4800
 $Comp
-L WS2812-2020:WS2812-2020 U?
+L pop-badge-rescue:WS2812-2020-WS2812-2020 U?
 U 1 1 617EF704
 P 4250 4800
@@
 	6250 4800 6450 4800
 $Comp
-L WS2812-2020:WS2812-2020 U?
+L pop-badge-rescue:WS2812-2020-WS2812-2020 U?
 U 1 1 617EF719
 P 5650 4800
@@
 $EndComp
 $Comp
-L WS2812-2020:WS2812-2020 U?
+L pop-badge-rescue:WS2812-2020-WS2812-2020 U?
 U 1 1 617EF72D
 P 7050 4800
@@
 $EndComp
 $Comp
-L WS2812-2020:WS2812-2020 U?
+L pop-badge-rescue:WS2812-2020-WS2812-2020 U?
 U 1 1 617EF744
 P 8450 4800
@@
 	3450 5950 3650 5950
 $Comp
-L WS2812-2020:WS2812-2020 U?
+L pop-badge-rescue:WS2812-2020-WS2812-2020 U?
 U 1 1 617F25BD
 P 2850 5950
@@
 	4850 5950 5050 5950
 $Comp
-L WS2812-2020:WS2812-2020 U?
+L pop-badge-rescue:WS2812-2020-WS2812-2020 U?
 U 1 1 617F25D2
 P 4250 5950
@@
 	6250 5950 6450 5950
 $Comp
-L WS2812-2020:WS2812-2020 U?
+L pop-badge-rescue:WS2812-2020-WS2812-2020 U?
 U 1 1 617F25E7
 P 5650 5950
@@
 $EndComp
 $Comp
-L WS2812-2020:WS2812-2020 U?
+L pop-badge-rescue:WS2812-2020-WS2812-2020 U?
 U 1 1 617F25FB
 P 7050 5950
@@
 $EndComp
 $Comp
-L WS2812-2020:WS2812-2020 U?
+L pop-badge-rescue:WS2812-2020-WS2812-2020 U?
 U 1 1 617F2612
 P 8450 5950
@@
 NoConn ~ 9050 5950
 $Comp
-L WS2812-2020:WS2812-2020 U?
+L pop-badge-rescue:WS2812-2020-WS2812-2020 U?
 U 1 1 617E1924
 P 8450 1200
@@
 	9050 1200 9600 1200
 $Comp
-L WS2812-2020:WS2812-2020 U?
+L pop-badge-rescue:WS2812-2020-WS2812-2020 U?
 U 1 1 617E18E4
 P 4250 1200
