File: pop-badge/pop-badge.sch (KiCad schematic (older format))
At the start: 13 parts, among them J1 Conn_01x06, Q1 S9013, Q2 AO3400A, U26 Pico

Commit message: remove button again
Parts:
- removed J1: Conn_01x06, Connector_PinHeader_2.54mm:PinHeader_1x06_P2.54mm_Vertical, symbol Connector_Generic:Conn_01x06
- removed R55: 200, Resistor_SMD:R_0603_1608Metric_Pad1.05x0.95mm_HandSolder, symbol Device:R
- removed S1: TS-1187A-B-A-B, footprints:SW_TS-1187A-B-A-B, symbol TS-button:TS-1187A-B-A-B
- added J1: Conn_01x05, Connector_PinHeader_2.54mm:PinHeader_1x05_P2.54mm_Vertical, symbol Connector_Generic:Conn_01x05
Connections:
- net labels removed: Button
- wire segments 25 -> 22
- no-connect marks 37 -> 38
Changed lines of the file:
@@
 Wire Wire Line
 	4150 4900 4150 5000
-Text GLabel 5400 3900 2    50   Input ~ 0
-Button
 $Comp
-L Device:R R55
-U 1 1 615CA836
-P 5400 4850
-F 0 "R55" H 5470 4896 50  0000 L CNN
-F 1 "200" H 5470 4805 50  0000 L CNN
-F 2 "Resistor_SMD:R_0603_1608Metric_Pad1.05x0.95mm_HandSolder" V 5330 4850 50  0001 C CNN
-F 3 "~" H 5400 4850 50  0001 C CNN
-F 4 "0603" H 5400 4850 50  0001 C CNN "JLC"
-	1    5400 4850
-	1    0    0    -1
-$EndComp
-$Comp
-L power:GND #PWR0103
-U 1 1 615CAE29
-P 5400 5000
-F 0 "#PWR0103" H 5400 4750 50  0001 C CNN
-F 1 "GND" H 5405 4827 50  0000 C CNN
-F 2 "" H 5400 5000 50  0001 C CNN
-F 3 "" H 5400 5000 50  0001 C CNN
-	1    5400 5000
-	1    0    0    -1
-$EndComp
-Wire Wire Line
-	5400 3900 5400 4100
-$Comp
-L Connector_Generic:Conn_01x06 J1
-U 1 1 615CEC6A
+L Connector_Generic:Conn_01x05 J1
+U 1 1 616045CF
 P 1600 950
-F 0 "J1" H 1680 942 50  0000 L CNN
-F 1 "Conn_01x06" H 1680 851 50  0000 L CNN
-F 2 "Connector_PinHeader_2.54mm:PinHeader_1x06_P2.54mm_Vertical" H 1600 950 50  0001 C CNN
+F 0 "J1" H 1680 992 50  0000 L CNN
+F 1 "Conn_01x05" H 1680 901 50  0000 L CNN
+F 2 "Connector_PinHeader_2.54mm:PinHeader_1x05_P2.54mm_Vertical" H 1600 950 50  0001 C CNN
 F 3 "~" H 1600 950 50  0001 C CNN
 	1    1600 950
 	1    0    0    -1
 $EndComp
-Text GLabel 1200 1250 0    50   Input ~ 0
-Button
-Text GLabel 5100 2450 2    50   Input ~ 0
-Button
-Wire Wire Line
-	5100 2450 4850 2450
-Wire Wire Line
-	1400 1250 1200 1250
-$Comp
-L TS-button:TS-1187A-B-A-B S1
-U 1 1 615D35C1
-P 5400 4400
-F 0 "S1" V 5354 4511 50  0000 L CNN
-F 1 "TS-1187A-B-A-B" V 5445 4511 50  0000 L CNN
-F 2 "footprints:SW_TS-1187A-B-A-B" H 5400 4400 50  0001 L BNN
-F 3 "" H 5400 4400 50  0001 L BNN
-F 4 "A0" H 5400 4400 50  0001 L BNN "PARTREV"
-F 5 "XKB Industrial Precision" H 5400 4400 50  0001 L BNN "MANUFACTURER"
-F 6 "1.5mm" H 5400 4400 50  0001 L BNN "MAXIMUM_PACKAGE_HEIGHT"
-F 7 "Manufacturer Recommendations" H 5400 4400 50  0001 L BNN "STANDARD"
-F 8 "C318884" H 5400 4400 50  0001 C CNN "JLC"
-	1    5400 4400
-	0    1    1    0
-$EndComp
+NoConn ~ 4850 2450
 $EndSCHEMATC

Commit message: add rescue lib
Parts:
- Q2: symbol AO3400a:AO3400A -> pop-badge-rescue:AO3400A-AO3400a
Changed lines of the file:
@@
 	3300 4600 3350 4600
 $Comp
-L AO3400a:AO3400A Q2
+L pop-badge-rescue:AO3400A-AO3400a Q2
 U 1 1 6158FC09
 P 4050 4500

Commit message: change footprint for npn slightly
Parts:
- Q1: footprint Package_TO_SOT_SMD:SOT-23 -> Package_TO_SOT_SMD:SOT-23_Handsoldering; symbol Transistor_BJT:BC818 -> Transistor_BJT:MMBTA42
Changed lines of the file:
@@
 	2250 4100 2250 4300
 $Comp
-L Transistor_BJT:BC818 Q?
+L Transistor_BJT:MMBTA42 Q?
 U 1 1 61BDB59D
 P 2150 4500
@@
 F 0 "Q1" H 2341 4546 50  0000 L CNN
 F 1 "S9013" H 2341 4455 50  0000 L CNN
-F 2 "Package_TO_SOT_SMD:SOT-23" H 2350 4425 50  0001 L CIN
+F 2 "Package_TO_SOT_SMD:SOT-23_Handsoldering" H 2350 4425 50  0001 L CIN
 F 3 "" H 2150 4500 50  0001 L CNN
 F 4 "C6749" H 2150 4500 50  0001 C CNN "JLC"
